Commit message: add pointcloud_to_laserscan

File: src/autoaim/rm_gimbal_description/urdf/rm_gimbal.urdf.xacro (robot description, xacro)
@@ -4,5 +4,5 @@
   <xacro:arg name="xyz" default="0.10 0 0.05" />
   <xacro:arg name="rpy" default="0 0 0" />
-  <link name="map" />
+  <link name="base_link" />
   <link name="gimbal_link" />
   <joint name="gimbal_joint" type="floating">
